Commit message: fix urdf bug

File: eagerx_demo/task/assets/bolt-template.urdf (robot description, URDF)
Before this commit: robot bolt, 1 links, 0 joints
Links:
- link baseLink: geometry collision mesh filename=bolt_centered.stl scale=0.0035 0.0035 0.0035; visual mesh filename=bolt_centered.stl scale=0.0035 0.0035 0.0035

File: eagerx_demo/task/assets/hollow_cylinder_L50R24T11H13-template.urdf (robot description, URDF)
Before this commit: robot box, 1 links, 0 joints
Links:
- link baseLink: geometry collision mesh filename=hollow_cylinder_L50R24T11H13.stl scale=0.001 0.001 0.0005; visual mesh filename=hollow_cylinder_L50R24T11H13.stl scale=0.001 0.001 0.0005
